File: KiCad/Ver1/GPIODriverVer1/OutputDrive.sch (KiCad schematic (older format))
At the start: 104 parts

Commit message: Save point Ver1 design.
Parts:
- D1, D13, D14, D15, D16, D17, D18, D19, D2, D20, D3, D4, D5, D6, D7, D8: renamed from D?; footprint (none) -> Diode_SMD:D_0603_1608Metric_Pad1.05x0.95mm_HandSolder
- D10, D11, D12, D21, D22, D23, D24, D9: renamed from D?; footprint (none) -> Diode_SMD:D_SOT-23_ANK
- F1, F2, F3, F4, F5, F6, F7, F8: renamed from F?; footprint (none) -> Resistor_SMD:R_0603_1608Metric
- Q1, Q13, Q14, Q15, Q16, Q2, Q3, Q4: renamed from Q?; footprint (none) -> Package_TO_SOT_SMD:SOT-723; symbol Device:Q_NPN_BCE -> Transistor_BJT:DTC143E
- Q11, Q17, Q19, Q21, Q23, Q5, Q7, Q9: renamed from Q?; footprint Package_TO_SOT_SMD:SOT-23 -> Package_TO_SOT_SMD:SOT-323_SC-70
- R17, R18, R19, R20, R21, R22, R23, R24, R25, R26, R27, R28, R29, R30, R31, R32, R33, R34, R35, R36, R37, R38, R39, R40, R41, R42, R43, R44, R45, R46, R47, R48, R49, R50, R51, R52, R53, R54, R55, R56, R57, R58, R59, R60, R61, R62, R63, R64: renamed from R?; footprint (none) -> Resistor_SMD:R_0402_1005Metric
- gave numbers to parts that had none: 8
Connections:
- net GND: now also Q1.2 (E), Q13.2 (E), Q14.2 (E), Q15.2 (E), Q16.2 (E), Q2.2 (E), Q3.2 (E), Q4.2 (E); no longer Q1.3 (E), Q13.3 (E), Q14.3 (E), Q15.3 (E), Q16.3 (E), Q2.3 (E), Q3.3 (E), Q4.3 (E)
- net at R25.1: now also Q1.3 (C); no longer Q1.2 (C)
- net at R26.1: now also Q2.3 (C); no longer Q2.2 (C)
- net at R27.1: now also Q3.3 (C); no longer Q3.2 (C)
- net at R28.1: now also Q4.3 (C); no longer Q4.2 (C)
- net at R49.1: now also Q13.3 (C); no longer Q13.2 (C)
- net at R50.1: now also Q14.3 (C); no longer Q14.2 (C)
- net at R51.1: now also Q15.3 (C); no longer Q15.2 (C)
- net at R52.1: now also Q16.3 (C); no longer Q16.2 (C)
