File: KiCad/Ver1/GPIODriverVer1/GPIODriverVer1.sch (KiCad schematic (older format))
At the start: 4 parts

Commit message: Updated schematic to include input/output buffers. Added connections for shift registers.
Parts:
- removed J?: Conn_01x08_Female, symbol Connector:Conn_01x08_Female
- removed U?: 74HC595, symbol 74xx:74HC595
- added J?: Conn_01x21_Male, symbol Connector:Conn_01x21_Male
- added R? (x2): 10k, symbol Device:R_US
- added R? (x13): 100, symbol Device:R_US
- added U? (x2): 74HC595_Nexperia, symbol 74xx:74HC595_Nexperia
- added U? (x2): 74HC244, symbol 74xx:74HC244
- U?: symbol 74HC165:74HC165 -> GPIODriverVer1-rescue:74HC165-74HC165
Connections:
- net labels added: GND, GPIO_CLK, GPIO_Sense_CS, GPIO_Sense_DI, GPIO_Sense_DO, GPIO_Sense_Load, GPIO_Sink_DI, GPIO_Sink_DO, GPIO_Sink_LAT, GPIO_Sink_OE, GPIO_Source_DI, GPIO_Source_DO, GPIO_Source_LAT, GPIO_Source_OE, SR_CLK, SenseDriver_CS, SenseDriver_DataIn, SenseDriver_DataOut, SenseDriver_Load, SinkDriver_DataIn, SinkDriver_DataOut, SinkDriver_LAT, SinkDriver_OE, SrcDriver_DataIn, SrcDriver_DataOut, SrcDriver_LAT, SrcDriver_OE, VCC, VDrive
- wire segments 39 -> 224
Other:
- moved on the sheet: J?

Commit message: Save point Ver1 design.
Parts:
- removed J?: Conn_01x21_Male, symbol Connector:Conn_01x21_Male
- added J1: Conn_01x22_Male, Connector_PinHeader_2.54mm:PinHeader_2x11_P2.54mm_Vertical, symbol Connector:Conn_01x22_Male
- added R14: 100, Resistor_SMD:R_0402_1005Metric, symbol Device:R_US
- added U3: NCV8452, Package_TO_SOT_SMD:SOT-223, symbol NCV8452:NCV8452
- J2: renamed from J?; footprint (none) -> Connector_PinHeader_2.54mm:PinHeader_1x08_P2.54mm_Horizontal
- R1, R10, R11, R12, R13, R15, R16, R2, R3, R4, R5, R6, R7, R8, R9: renamed from R?; footprint (none) -> Resistor_SMD:R_0402_1005Metric
- U1, U2: renamed from U?; footprint (none) -> Package_SO:TSSOP-20_4.4x6.5mm_P0.65mm
- U4, U5: renamed from U?; footprint (none) -> Package_SO:TSSOP-16_4.4x5mm_P0.65mm; symbol 74xx:74HC595_Nexperia -> GPIODriverVer1-rescue:74HC595_Nexperia-74xx
- U6: renamed from U?; footprint (none) -> Package_SO:TSSOP-16_4.4x5mm_P0.65mm
Connections:
- net GND: now also J1.11 (Pin_11), J1.16 (Pin_16), J1.2 (Pin_2), J1.21 (Pin_21), J1.4 (Pin_4), J1.6 (Pin_6), U3.2 (GND); no longer U2.15 (2A1)
- net VCC: now also J1.3 (Pin_3)
- net VDrive: now also U3.1 (OUT)
- net PowerEnable: now reaches U2.5 (2Y1)
- net PowerEnable: now also U3.3 (CTRL)
- net at R5.2: now also J1.10 (Pin_10)
- net at R6.2: now also J1.12 (Pin_12)
- net at R7.2: now also J1.13 (Pin_13)
- net at R8.2: now also J1.14 (Pin_14)
- net at R9.2: now also J1.15 (Pin_15)
- net at R10.2: now also J1.17 (Pin_17)
- net at R11.2: now also J1.18 (Pin_18)
- net at R12.2: now also J1.19 (Pin_19)
- net at R13.2: now also J1.20 (Pin_20)
- net at R1.2: now also J1.5 (Pin_5)
- net at R2.2: now also J1.7 (Pin_7)
- net at R3.2: now also J1.8 (Pin_8)
- net at R4.2: now also J1.9 (Pin_9)
- new net: J1.22 (Pin_22), R14.2
- new net GPIO_PWR_EN: R14.1, U2.15 (2A1)
- new net V+: J1.1 (Pin_1), U3.4 (VD)
Other:
- moved on the sheet: J2, R15, R16, U1, U2, U4, U5, U6

Commit message: Planned a little more of the Version 2 board.
Parts:
- U3: symbol NCV8452:NCV8452 -> GPIODriverVer1-rescue:NCV8452-NCV8452
Changed lines of the file:
@@
 	1700 1050 2550 1050
 $Comp
-L NCV8452:NCV8452 U3
+L GPIODriverVer1-rescue:NCV8452-NCV8452 U3
 U 1 1 5CC26F8D
 P 8200 1300
